File: kicad/ring.kicad_sch (KiCad schematic)
At the start: 2 parts

Commit message: init
Parts:
- added J1: Conn_01x02, Connector_Phoenix_MSTB:PhoenixContact_MSTBVA_2,5_2-G_1x02_P5.00mm_Vertical, symbol Connector_Generic:Conn_01x02
- added P1: USB_C_Plug_USB2.0, symbol Connector:USB_C_Plug_USB2.0
- added U1: ESP32-WROOM-E, PCM_Espressif:ESP32-WROOM-32E, symbol PCM_Espressif:ESP32-WROOM-E
Connections:
- net GND: now reaches PS1.3 (-Vout)
- net GND: now also P1.A1 (GND), P1.A12 (GND), P1.B1 (GND), P1.B12 (GND), P1.S1 (SHIELD), U1.1 (GND), U1.15 (GND), U1.38 (GND)
- net AC: no longer names the net of F1.1
- net AC: now also J1.2 (Pin_2)
- new net: P1.A4 (VBUS), P1.A9 (VBUS), P1.B4 (VBUS), P1.B9 (VBUS)

Commit message: init
Parts:
- removed F1: Fuse, Fuse:Fuse_Bourns_MF-RG300, symbol Device:Fuse
- removed J1: Conn_01x02, Connector_Phoenix_MSTB:PhoenixContact_MSTBVA_2,5_2-G_1x02_P5.00mm_Vertical, symbol Connector_Generic:Conn_01x02
- removed P1: USB_C_Plug_USB2.0, symbol Connector:USB_C_Plug_USB2.0
- removed PS1: HLK-PM01, Converter_ACDC:Converter_ACDC_Hi-Link_HLK-PMxx, symbol Converter_ACDC:HLK-PM01
Other:
- added sheet Supply (supply.kicad_sch)
- moved on the sheet: U1
