File: kicad/supply.kicad_sch (KiCad schematic)
At the start: 18 parts, among them J1 Conn_01x02, P1 USB_C_Plug_USB2.0, U2 CP2102N-Axx-xQFN20

Commit message: init
Parts:
- removed U2: CP2102N-Axx-xQFN20, Package_DFN_QFN:QFN-20-1EP_3x3mm_P0.45mm_EP1.6x1.6mm, symbol Interface_USB:CP2102N-Axx-xQFN20
- added U3: CP2102N-Axx-xQFN28, Package_DFN_QFN:QFN-28-1EP_5x5mm_P0.5mm_EP3.35x3.35mm, symbol Interface_USB:CP2102N-Axx-xQFN28
Connections:
- net +3.3V: now also U3.6 (VDD), U3.7 (VREGIN)
- net GND: now also U3.29 (GND), U3.3 (GND)
- net RXD: now also U3.25 (RXD)
- net TXD: now also U3.26 (TXD)
- net at P1.A6 (D+): now also U3.4 (D+)
- net at P1.A7 (D-): now also U3.5 (D-)
- net at R2.2, R3.1: now also U3.8 (VBUS)
- net at R6.1: now also U3.11 (~{SUSPEND})
- net at R5.1: now also U3.24 (~{RTS})
Changed lines of the file:
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@@
+	(wire
+		(pts
+			(xy 121.92 177.8) (xy 121.92 180.34)
+		)
+		(stroke
+			(width 0)
+			(type default)
+		)
+	)
 	(wire
 		(pts
@@
 		(shape input)
 		(at 146.05 119.38 0)
-		(fields_autoplaced yes)
 		(effects
 			(font
@@
 		(shape input)
 		(at 146.05 116.84 0)
-		(fields_autoplaced yes)
 		(effects
 			(font
@@
 	(symbol
 		(lib_id "power:GND")
-		(at 121.92 167.64 0)
+		(at 121.92 180.34 0)
 		(unit 1)
 		(exclude_from_sim no)
@@
 		(fields_autoplaced yes)
 		(property "Reference" "#PWR012"
-			(at 121.92 173.99 0)
+			(at 121.92 186.69 0)
 			(effects
 				(font
@@
 		)
 		(property "Value" "GND"
-			(at 121.92 172.085 0)
+			(at 121.92 184.785 0)
 			(effects
 				(font
@@
 		)
 		(property "Footprint" ""
-			(at 121.92 167.64 0)
+			(at 121.92 180.34 0)
 			(effects
 				(font
@@
 		)
 		(property "Datasheet" ""
-			(at 121.92 167.64 0)
+			(at 121.92 180.34 0)
 			(effects
 				(font
@@
 		)
 		(property "Description" "Power symbol creates a global label with name \"GND\" , ground"
-			(at 121.92 167.64 0)
+			(at 121.92 180.34 0)
 			(effects
 				(font
@@
 	)
 	(symbol
+		(lib_id "Interface_USB:CP2102N-Axx-xQFN28")
+		(at 121.92 144.78 0)
+		(unit 1)
+		(exclude_from_sim no)
+		(in_bom yes)
+		(on_board yes)
+		(dnp no)
+		(fields_autoplaced yes)
+		(property "Reference" "U3"
+			(at 124.1141 177.8 0)
+			(effects
+				(font
+					(size 1.27 1.27)
+				)
+				(justify left)
+			)
+		)
+		(property "Value" "CP2102N-Axx-xQFN28"
+			(at 124.1141 180.34 0)
+			(effects
+				(font
+					(size 1.27 1.27)
+				)
+				(justify left)
+			)
+		)
+		(property "Footprint" "Package_DFN_QFN:QFN-28-1EP_5x5mm_P0.5mm_EP3.35x3.35mm"
+			(at 154.94 176.53 0)
+			(effects
+				(font
+					(size 1.27 1.27)
+				)
+				(hide yes)
+			)
+		)
+		(property "Datasheet" "https://www.silabs.com/documents/public/data-sheets/cp2102n-datasheet.pdf"
+			(at 123.19 163.83 0)
+			(effects
+				(font
+					(size 1.27 1.27)
+				)
+				(hide yes)
+			)
+		)
+		(property "Description" "USB to UART master bridge, QFN-28"
+			(at 121.92 144.78 0)
+			(effects
+				(font
+					(size 1.27 1.27)
+				)
+				(hide yes)
+			)
+		)
+		(pin "2"
+		)
+		(pin "23"
+		)
+		(pin "24"
+		)
+		(pin "27"
+		)
+		(pin "20"
+		)
+		(pin "4"
+		)
+		(pin "8"
+		)
+		(pin "1"
+		)
+		(pin "6"
+		)
+		(pin "7"
+		)
+		(pin "11"
+		)
+		(pin "18"
+		)
+		(pin "22"
+		)
+		(pin "17"
+		)
+		(pin "12"
+		)
+		(pin "21"
+		)
+		(pin "29"
+		)
+		(pin "3"
+		)
+		(pin "9"
+		)
+		(pin "25"
+		)
+		(pin "19"
+		)
+		(pin "10"
+		)
+		(pin "26"
+		)
+		(pin "15"
+		)
+		(pin "28"
+		)
+		(pin "14"
+		)
+		(pin "16"
+		)
+		(pin "5"
+		)
+		(pin "13"
+		)
+		(instances
+			(project ""
+				(path "/1f81e754-27ae-476e-a47b-63ee7b14e765/d9c1ca1f-9609-4271-8008-f6dce5bf188a"
+					(reference "U3")
+					(unit 1)
+				)
+			)
+		)
+	)
+	(symbol
 		(lib_id "Device:R")
 		(at 104.14 140.97 0)
@@
 					(unit 1)
 				)
-			)
-		)
-	)
-	(symbol
-		(lib_id "Interface_USB:CP2102N-Axx-xQFN20")
-		(at 121.92 139.7 0)
-		(unit 1)
-		(exclude_from_sim no)
-		(in_bom yes)
-		(on_board yes)
-		(dnp no)
-		(fields_autoplaced yes)
-		(property "Reference" "U2"
-			(at 124.1141 167.005 0)
-			(effects
-				(font
-					(size 1.27 1.27)
-				)
-				(justify left)
-			)
-		)
-		(property "Value" "CP2102N-Axx-xQFN20"
-			(at 124.1141 169.545 0)
-			(effects
-				(font
-					(size 1.27 1.27)
-				)
-				(justify left)
-			)
-		)
-		(property "Footprint" "Package_DFN_QFN:QFN-20-1EP_3x3mm_P0.45mm_EP1.6x1.6mm"
-			(at 153.67 166.37 0)
-			(effects
-				(font
-					(size 1.27 1.27)
-				)
-				(hide yes)
-			)
-		)
-		(property "Datasheet" "https://www.silabs.com/documents/public/data-sheets/cp2102n-datasheet.pdf"
-			(at 123.19 158.75 0)
-			(effects
-				(font
-					(size 1.27 1.27)
-				)
-				(hide yes)
-			)
-		)
-		(property "Description" "USB to UART master bridge, QFN-20"
-			(at 121.92 139.7 0)
-			(effects
-				(font
-					(size 1.27 1.27)
-				)
-				(hide yes)
-			)
-		)
-		(property "LCSC" "C969913"
-			(at 124.1141 167.005 0)
-			(effects
-				(font
-					(size 1.27 1.27)
-				)
-				(hide yes)
-			)
-		)
-		(pin "4"
-		)
-		(pin "20"
-		)
-		(pin "8"
-		)
-		(pin "18"
-		)
-		(pin "15"
-		)
-		(pin "7"
-		)
-		(pin "6"
-		)
-		(pin "1"
-		)
-		(pin "2"
-		)
-		(pin "17"
-		)
-		(pin "3"
-		)
-		(pin "14"
-		)
-		(pin "19"
-		)
-		(pin "16"
-		)
-		(pin "10"
-		)
-		(pin "5"
-		)
-		(pin "11"
-		)
-		(pin "13"
-		)
-		(pin "12"
-		)
-		(pin "21"
-		)
-		(pin "9"
-		)
-		(instances
-			(project "ring"
-				(path "/1f81e754-27ae-476e-a47b-63ee7b14e765/d9c1ca1f-9609-4271-8008-f6dce5bf188a"
-					(reference "U2")
-					(unit 1)
-				)
